Commit message: removed mesh file on .urdf files

File: urdf/two_link_fk.urdf (robot description, URDF)
Before this commit: robot two_link_robot, 4 links, 3 joints
Links:
- link tibia: geometry visual cylinder length=0.005 radius=0.0025

File: urdf/two_link_ik.urdf (robot description, URDF)
Before this commit: robot two_link_robot, 4 links, 3 joints
Links:
- link ee_link: geometry collision box size=0.01 0.01 0.01; visual cylinder length=0.005 radius=0.0025
